File: Ears 0603.brd (EAGLE design)
At the start: 19.2 x 108.4 mm, 75 parts, among them IC1 OPA1641, IC2 LM324D, IC3 LM324D, J1 PJ301_THONKICONN6, J2 PJ301_THONKICONN6, J3 PJ301_THONKICONN6, J4 PJ301_THONKICONN6

Commit message: Add files via upload
Parts:
- moved R26 0.60 mm to (15.4, 17.4)
- moved C13 0.50 mm to (2.13, 17.4)
- moved R25 0.50 mm to (13.5, 17.4)
- moved R24 0.40 mm to (11.7, 17.4)
- moved C12 0.35 mm to (4.13, 17.4)
- moved R23 0.30 mm to (9.88, 17.4)
- moved C11 0.20 mm to (6.08, 17.4)
- moved R27 0.10 mm to (8.01, 17.4)
Routing:
- net N$18: track 13.7 -> 14.6 mm
- net N$19: track 21.8 -> 22.4 mm
- net AMP_OUT: track 53.9 -> 53.3 mm
